File: Button.brd (EAGLE design)
At the start: 22.7 x 20.1 mm, 27 parts, among them U1 NRF51822-QFAB-R7, X1 16MHz

Commit message: Adding Brd and such files for Button board update
Parts:
- removed JP1: (no value), SparkFun-v5:1X04-1.27MM
- added K1: 665104131822, Wurth_Elektronik_Electromechanic_Wire_to_Board_Connectors_rev15c:665104131822
- LED1: device apdm_alt:KINGBRITE_RGBLED_1.6X1.26 -> rgb-led-separate:LED-3528
- R1, R2: value 10k -> (none); device rcl_custom:.0402-C-NOSILK -> adafruit:R0402
- moved R1 4.05 mm to (17.4, 1.42), turned to 90 degrees
- moved R2 3.48 mm to (8.48, 3.35)
- moved R5 1.91 mm to (3.56, 13.5)
- moved LED1 1.15 mm to (2.92, 10.2)
- moved B1 0.94 mm to (8.00, 11.0)
- moved C5 0.86 mm to (4.83, 4.93)
- moved R3 0.72 mm to (5.84, 8.00)
- moved R4 0.18 mm to (6.22, 9.91)
- moved C1 0.13 mm to (7.11, 5.71)
Connections:
- removed net SWDCLK: JP1.3, R1.1, U1.24
- removed net SWDIO: JP1.2, R2.1, U1.23
- new net N$11: K1.2, R2.1, U1.23
- new net N$14: R2.2
- new net N$9: K1.3, R1.2, U1.24
- net GND: now also K1.4, R1.1; no longer JP1.4, R1.2
- net N$1: now also U1.5; no longer U1.4
- net N$2: now also U1.6; no longer U1.5
- net N$3: now also U1.7; no longer U1.6
- net N$4: now also LED1.6; no longer LED1.3
- net N$5: now also LED1.5; no longer LED1.4
- net N$7: now also LED1.4; no longer LED1.1
- net VDD: now also K1.1, LED1.1, LED1.3; no longer JP1.1, R2.2
Routing:
- net N$11: track 0.00 -> 16.9 mm
- net N$9: track 0.00 -> 9.79 mm
- net VDD: track 51.8 -> 46.6 mm, vias 2 -> 3
- net SWDIO: track 3.62 -> 0.00 mm
- net SWDCLK: track 3.49 -> 0.00 mm
- net N$4: track 0.99 -> 3.42 mm
- net N$1: track 5.19 -> 6.60 mm
- net N$7: track 0.98 -> 2.01 mm
- net N$5: track 1.27 -> 1.79 mm
- net GND: vias 46 -> 65
Other:
- board size 22.7 x 20.1 mm -> 22.8 x 27 mm

Commit message: lasted version of brd and such
Parts:
- moved K1 4.20 mm to (16.7, 3.20), flipped to the bottom, turned to 270 degrees
- moved R2 4.13 mm to (11.7, 0.81), flipped to the bottom
- moved R1 3.03 mm to (14.4, 0.81), flipped to the bottom, turned to 180 degrees
- moved B1 0.78 mm to (8.26, 10.2)
- moved C4 0.06 mm to (15.2, 5.99)
Routing:
- net N$11: track 16.9 -> 9.96 mm, vias 0 -> 2
- net N$9: track 9.79 -> 7.64 mm, vias 0 -> 1
- net VDD: track 46.6 -> 44.7 mm, vias 3 -> 2
- net GND: vias 65 -> 66
Other:
- board size 22.8 x 27 mm -> 22.8 x 27.1 mm
