File: Button.sch (EAGLE design)
At the start: 26 parts, among them U1 NRF51822-QFAB-R7, X1 16MHz

Commit message: Adding Brd and such files for Button board update
Parts:
- removed JP1: (no value), SparkFun-v5:M041.27MM
- added K1: 665104131822, Wurth_Elektronik_Electromechanic_Wire_to_Board_Connectors_rev15c:665104131822
- LED1: device apdm_alt:LED_RGB_COMMON_ANODE-1.6X1.26 -> rgb-led-separate:LED-RGB-SEPARATE-3528
- R1, R2: value 10k -> (none); device rcl_custom:R-US_0402-C-NOSILK -> adafruit:R-US_R0402
Connections:
- removed net SWDCLK: JP1.3, R1.1, U1.SWDCLK
- removed net SWDIO: JP1.2, R2.1, U1.SWDIO/NRESET
- new net N$11: K1.2, R2.1, U1.SWDIO/NRESET
- new net N$14: R2.2
- new net N$9: K1.3, R1.2, U1.SWDCLK
- net GND: now also K1.4, R1.1; no longer JP1.4, R1.2
- net N$1: now also U1.P0.01/AIN2; no longer U1.P0.00/AREF0
- net N$2: now also U1.P0.02/AIN3; no longer U1.P0.01/AIN2
- net N$3: now also U1.P0.03/AIN4; no longer U1.P0.02/AIN3
- net N$4: now also LED1B.K; no longer LED1.RK
- net N$5: now also LED1R.K; no longer LED1.GK
- net N$7: now also LED1G.K; no longer LED1.BK
- net VDD: now also K1.1, LED1B.A, LED1G.A, LED1R.A; no longer JP1.1, LED1.COMMON_ANODE, R2.2
Other:
- moved on the sheet: U1
